Commit message: Made changes in robot desc to support gazebo classic

File: turtlebot4_description/urdf/sensors/oakd.urdf.xacro (robot description, xacro)
@@ -1,5 +1,5 @@
 <?xml version="1.0"?>
 <robot xmlns:xacro="http://ros.org/wiki/xacro">
-<xacro:macro name="oakd" params="name:=oakd parent_link *origin model:=pro">
+<xacro:macro name="oakd" params="name:=oakd parent_link gazebo *origin model:=pro">
   <xacro:include filename="$(find irobot_create_description)/urdf/common_properties.urdf.xacro"/>
   <xacro:property name="mass"       value="0.061"/>
@@ -99,21 +99,25 @@
   <!-- Gazebo links and joints -->
   <gazebo reference="${name}_rgb_camera_frame">
-    <sensor name="rgbd_camera" type="rgbd_camera">
-      <camera>
-        <horizontal_fov>1.25</horizontal_fov>
-        <image>
-          <width>320</width>
-          <height>240</height>
-        </image>
-        <clip>
-          <near>0.3</near>
-          <far>100</far>
-        </clip>
-        <optical_frame_id>${name}_rgb_camera_optical_frame</optical_frame_id>
-      </camera>
-      <always_on>1</always_on>
-      <update_rate>30</update_rate>
-      <visualize>true</visualize>
-    </sensor>
+    <xacro:if value="${gazebo == 'ignition'}">
+      <sensor name="rgbd_camera" type="rgbd_camera">
+        <camera>
+          <horizontal_fov>1.25</horizontal_fov>
+          <image>
+            <width>320</width>
+            <height>240</height>
+          </image>
+          <clip>
+            <near>0.3</near>
+            <far>100</far>
+          </clip>
+          <optical_frame_id>${name}_rgb_camera_optical_frame</optical_frame_id>
+        </camera>
+        <always_on>1</always_on>
+        <update_rate>30</update_rate>
+        <visualize>true</visualize>
+      </sensor>
+    </xacro:if>
+    <xacro:if value="${gazebo == 'classic'}">
+    </xacro:if>
     <xacro:material_darkgray/>
   </gazebo>

File: turtlebot4_description/urdf/sensors/rplidar.urdf.xacro (robot description, xacro)
@@ -30,10 +30,44 @@
   </link>
   <gazebo reference="${name}_link">
-    <xacro:ray_sensor sensor_name="${name}" gazebo="${gazebo}"
-                  update_rate="62.0" visualize="1"
-                  h_samples="640" h_res="1.0" h_min_angle="${-pi}" h_max_angle="${pi}"
-                  r_min="0.164" r_max="12.0" r_res="0.01">
-                  <plugin name="dummy" filename="dummyfile"></plugin>
-    </xacro:ray_sensor>
+    <xacro:if value="${gazebo == 'ignition'}">
+      <xacro:ray_sensor sensor_name="${name}" gazebo="${gazebo}"
+                    update_rate="62.0" visualize="1"
+                    h_samples="640" h_res="1.0" h_min_angle="${-pi}" h_max_angle="${pi}"
+                    r_min="0.164" r_max="12.0" r_res="0.01">
+                    <plugin name="dummy" filename="dummyfile"></plugin>
+      </xacro:ray_sensor>
+    </xacro:if>
+    <xacro:if value="${gazebo == 'classic'}">
+      <sensor type="gpu_ray" name="{name}">
+        <pose>0 0 0.5 0 0 0</pose>
+        <visualize>true</visualize>
+        <update_rate>62.0</update_rate>
+        <ray>
+          <scan>
+            <horizontal>
+              <samples>640</samples>
+              <resolution>1</resolution>
+              <min_angle>${-pi}</min_angle>
+              <max_angle>${pi}</max_angle>
+            </horizontal>
+          </scan>
+          <range>
+            <min>0.164</min>
+            <max>12.0</max>
+            <resolution>0.01</resolution>
+          </range>
+          <!-- <noise>
+            <type>gaussian</type>
+            <mean>0.0</mean>
+            <stddev>0.01</stddev>
+          </noise> -->
+        </ray>
+        <plugin name="gazebo_ros_head_rplidar_controller" filename="libgazebo_ros_ray_sensor.so">
+          <topicName>scan</topicName>
+          <frameName>laser</frameName>
+          <output_type>sensor_msgs/LaserScan</output_type>
+        </plugin>
+      </sensor>
+    </xacro:if>
     <xacro:material_darkgray/>
   </gazebo>

File: turtlebot4_description/urdf/standard/turtlebot4.urdf.xacro (robot description, xacro)
@@ -98,5 +98,5 @@
     <origin xyz="${camera_mount_x_offset} ${camera_mount_y_offset} ${camera_mount_z_offset}"/>
   </xacro:camera_bracket>
-  <xacro:oakd model="pro" parent_link="oakd_camera_bracket">
+  <xacro:oakd model="pro" parent_link="oakd_camera_bracket" gazebo="$(arg gazebo)">
     <origin xyz="${oakd_pro_x_offset} ${oakd_pro_y_offset} ${oakd_pro_z_offset}"/>
   </xacro:oakd>
